File: hardware/hardware.kicad_pcb (KiCad board)
At the start: 2 copper layers, 55 x 33.8 mm, 19 parts, among them J1 6P6C - RJ11, J2 2.54mm Header, U1 HT9032D, Y1 3.58MHz

Commit message: tidy
Parts:
- C1, C3: value 0.01MFD -> 0.01uF
- C2: value 0.1MFD -> 0.1uF
- C6, C7: value 0.22MFD -> 0.22uF
Connections:
- net VDD renamed +5V
