File: hardware/hardware.kicad_sch (KiCad schematic)
At the start: 19 parts, among them J1 6P6C - RJ11, J2 2.54mm Header, U1 HT9032D, Y1 3.58MHz

Commit message: tidy
Parts:
- C1, C3: value 0.01MFD -> 0.01uF; JLCPCB Part (none) -> C109484; MFR.Part (none) -> MPP103J2G1305085LC
- C2: value 0.1MFD -> 0.1uF; JLCPCB Part (none) -> C84772; MFR.Part (none) -> CT4-0805B104K500F3
- C4, C5: JLCPCB Part (none) -> C94712; MFR.Part (none) -> CC4-0805N330J500F3
- C6, C7: value 0.22MFD -> 0.22uF; JLCPCB Part (none) -> C914540; MFR.Part (none) -> CBB21-224J-400V
- D1: JLCPCB Part (none) -> C266671; MFR.Part (none) -> 2W10G-E4/51
- J1: JLCPCB Part (none) -> C588140; MFR.Part (none) -> 520186646
- J2: JLCPCB Part (none) -> C32713271; MFR.Part (none) -> HX PZ2.54-1x5P ZZ
- R1, R2: JLCPCB Part (none) -> C2894668; MFR.Part (none) -> CR1/4W-200K±5%-ST52
- R3: JLCPCB Part (none) -> C2894673; MFR.Part (none) -> CR1/4W-22K±5%-ST52
- R4: JLCPCB Part (none) -> C2894650; MFR.Part (none) -> CR1/4W-10M±5%-ST52
- R5: JLCPCB Part (none) -> C120119; MFR.Part (none) -> CF1/4W-470KΩ±5% T
- R6: JLCPCB Part (none) -> C120085; MFR.Part (none) -> CF1/4W-18KΩ±5% T52
- R7: JLCPCB Part (none) -> C2894540; MFR.Part (none) -> CR1/4W-15K±5%-OT26
- U1: JLCPCB Part (none) -> C22397227; MFR.Part (none) -> HT9032D(LX)
- Y1: JLCPCB Part (none) -> C20617999; MFR.Part (none) -> X49SD358MSB2SC-1
